File: LEDPendant.kicad_pcb (KiCad board)
At the start: 2 copper layers, 34.3 x 78.7 mm, 34 parts, among them U1 nRF24LU1P, U2 APA-102, U3 APA-102, U4 APA-102, U5 APA-102, U6 APA-102, U7 APA-102, U8 LD1117S33TR, Y1 Crystal

Commit message: Another pass at the large board
Parts:
- added R10: 22k, Resistors_SMD:R_0805, F.Cu at (210.8, 125.1)
- added R11: 47k, Resistors_SMD:R_0805, F.Cu at (210.8, 103.5)
- added R8: 100k, Resistors_SMD:R_0805, F.Cu at (221.6, 97.2)
- added R9: 10k, Resistors_SMD:R_0805, F.Cu at (210.8, 146.7)
- added SW1: SPST, Buttons_Switches_SMD:SW_SPST_PTS645, F.Cu at (216.5, 143.5)
- added SW2: SPST, Buttons_Switches_SMD:SW_SPST_PTS645, F.Cu at (216.5, 121.9)
- added SW3: SPST, Buttons_Switches_SMD:SW_SPST_PTS645, F.Cu at (216.5, 100.3)
- C1, C10, C11, C2, C3, C4, C5, C6, C7, C8, C9, L1, L2, L3, R1, R2, R3, R4, R5, R6, R7, U1, Y1: moved to F.Cu
- moved R7 102.0 mm to (262.6, 138.4), turned to 0 degrees
- moved R5 94.2 mm to (266.5, 132.1), turned to 0 degrees
- moved C7 82.2 mm to (249.6, 132.1), turned to 0 degrees
- moved C5 81.8 mm to (237.5, 138.4)
- moved C11 81.6 mm to (242.0, 144.7), turned to 0 degrees
- moved C9 79.2 mm to (246.6, 138.4)
- moved R1 77.7 mm to (255.3, 138.4)
- moved R4 76.8 mm to (254.5, 144.7)
- moved R6 76.1 mm to (259.0, 138.4)
- moved C10 74.5 mm to (237.6, 144.7), turned to 0 degrees
- moved R2 72.4 mm to (262.9, 132.1)
- moved C6 71.9 mm to (245.6, 132.1)
- moved C8 69.9 mm to (241.9, 138.4)
- moved C3 67.8 mm to (230.6, 148.7), turned to 0 degrees
- moved R3 66.9 mm to (250.8, 144.7)
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Routing:
- net Net-(L1-Pad1): track 60.3 -> 0.00 mm
- net Net-(U1-Pad10): track 52.3 -> 0.00 mm, vias 1 -> 0
- net Net-(U1-Pad11): track 42.3 -> 0.00 mm, vias 1 -> 0
- net Net-(C3-Pad2): track 37.3 -> 0.00 mm
- net GND: track 35.6 -> 6.86 mm, vias 18 -> 4
- net Net-(R5-Pad2): track 23.6 -> 0.00 mm
- net Net-(C1-Pad1): track 23.6 -> 0.00 mm
- net Net-(R4-Pad2): track 23.3 -> 0.00 mm, vias 2 -> 0
- net Net-(U3-Pad2): track 27.4 -> 5.12 mm, vias 2 -> 0
- net Net-(U3-Pad1): track 24.4 -> 5.12 mm
- net Net-(L1-Pad2): track 16.4 -> 0.00 mm
- net Net-(C2-Pad2): track 15.2 -> 0.00 mm
- net Net-(C6-Pad1): track 13.7 -> 0.00 mm, vias 2 -> 0
- net Net-(R1-Pad1): track 13.5 -> 0.00 mm, vias 1 -> 0
- net VCC: track 16.6 -> 3.39 mm, vias 6 -> 2
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Other:
- board size 34.3 x 78.7 mm -> 95.9 x 55.9 mm

Commit message: More hand routing
Parts:
- ANT1, C10, C11, C4, C8, C9, L1, L2, L3, R1, R10, R11, R2, R4, R5, R6, R8, R9: moved to B.Cu
- moved C9 99.1 mm to (147.6, 143.5), turned to 270 degrees
- moved C11 97.2 mm to (147.6, 121.9)
- moved C10 91.8 mm to (147.6, 127.0), turned to 90 degrees
- moved R2 84.4 mm to (181.1, 111.3), turned to 180 degrees
- moved R6 81.1 mm to (181.1, 115.8), turned to 180 degrees
- moved R7 70.4 mm to (193.3, 126.5), turned to 180 degrees
- moved C5 63.0 mm to (177.5, 118.9), turned to 180 degrees
- moved C8 62.7 mm to (179.3, 135.4)
- moved C4 62.2 mm to (179.3, 131.8), turned to 180 degrees
- moved R3 60.4 mm to (199.4, 113.0), turned to 90 degrees
- moved C7 57.1 mm to (193.3, 122.9)
- moved R5 56.8 mm to (210.8, 120.9), turned to 90 degrees
- moved C6 53.6 mm to (193.3, 120.4)
- moved C1 51.8 mm to (186.7, 109.5), turned to 90 degrees
- moved R4 51.8 mm to (210.8, 116.8), turned to 90 degrees
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Routing:
- net Net-(L1-Pad2): track 0.00 -> 56.9 mm, vias 0 -> 1
- net Net-(L1-Pad1): track 0.00 -> 56.8 mm, vias 0 -> 1
- net Net-(C9-Pad1): track 0.00 -> 56.5 mm, vias 0 -> 1
- net Net-(R4-Pad2): track 0.00 -> 49.1 mm, vias 0 -> 1
- net Net-(R5-Pad2): track 0.00 -> 45.0 mm, vias 0 -> 1
- net VCC: track 3.39 -> 43.3 mm, vias 2 -> 11
- net Net-(R8-Pad2): track 0.00 -> 35.2 mm, vias 0 -> 1
- net GND: track 6.86 -> 40.9 mm
- net Net-(C3-Pad2): track 0.00 -> 22.4 mm
- net Net-(C2-Pad2): track 0.00 -> 20.7 mm
- net Net-(R4-Pad1): track 0.00 -> 12.8 mm, vias 0 -> 1
- net Net-(R5-Pad1): track 0.00 -> 12.2 mm, vias 0 -> 1
- net Net-(R2-Pad1): track 0.00 -> 9.39 mm, vias 0 -> 1
- net Net-(C1-Pad1): track 0.00 -> 8.70 mm
- net Net-(ANT1-Pad1): track 0.00 -> 7.83 mm
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
Commit message: Passing ERC/DRC
Parts:
- R2: moved to F.Cu
Routing:
- net Net-(R8-Pad2): track 35.2 -> 113.8 mm, vias 1 -> 3
- net Net-(C1-Pad1): track 8.70 -> 63.8 mm, vias 0 -> 1
- net GND: track 40.9 -> 92.7 mm, vias 4 -> 11
- net Net-(U1-Pad11): track 0.00 -> 45.2 mm
- net Net-(U1-Pad10): track 0.00 -> 41.7 mm
- net Net-(R9-Pad2): track 6.62 -> 14.6 mm
- net Net-(R11-Pad2): track 5.79 -> 13.7 mm
- net Net-(R10-Pad2): track 6.62 -> 12.4 mm
- net VCC: track 43.3 -> 46.3 mm, vias 11 -> 12
- net Net-(R2-Pad1): track 9.39 -> 9.15 mm, vias 1 -> 0

Commit message: Add cr2032 battery
Parts:
- added BATT_CR2032_MPD: VAL**, imciner2_Footprints:BATT_CR2032_MPD, F.Cu at (167.0, 111.8)
Routing:
- net +BATT: track 0.00 -> 12.8 mm, vias 0 -> 1
Changed lines of the file:
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@@
 (kicad_pcb (version 4) (host pcbnew "(2015-05-23 BZR 5679)-product")
   (general
-    (links 102)
+    (links 104)
     (no_connects 0)
-    (area 128.643919 92.95 232.778729 149.910001)
+    (area 119.000001 89.225 232.778729 149.910001)
     (thickness 1.6)
-    (drawings 4)
-    (tracks 300)
+    (drawings 6)
+    (tracks 305)
     (zones 0)
-    (modules 41)
+    (modules 42)
     (nets 44)
   )
@@
     (mod_text_size 1 1)
     (mod_text_width 0.15)
-    (pad_size 1.5 1.5)
-    (pad_drill 0.6)
+    (pad_size 3.29 3.29)
+    (pad_drill 0)
     (pad_to_mask_clearance 0)
     (aux_axis_origin 0 0)
@@
   (module antennes:Ant_Microchip_2_4G (layer B.Cu)
     (at 142.24 121.92 270)
-    (fp_text reference ANT1 (at 0 11.00074 270) (layer B.SilkS)
+    (fp_text reference ANT1 (at 0 8.89 270) (layer B.SilkS)
       (effects (font (size 1.23952 1.23952) (thickness 0.3048)) (justify mirror))
     )
@@
     (pad 3 smd rect (at 2.19964 -1.19888 90) (size 1.80086 1.39954) (layers F.Cu F.Paste F.Mask))
     (pad 4 smd rect (at -2.19964 -1.19888 90) (size 1.80086 1.39954) (layers F.Cu F.Paste F.Mask))
+  )
+  (module imciner2_Footprints:BATT_CR2032_MPD (layer F.Cu)
+    (at 167.005 111.76 90)
+    (fp_text reference BATT_CR2032_MPD (at -2.54 -2.54 90) (layer F.SilkS)
+      (effects (font (thickness 0.3048)))
+    )
+    (fp_text value VAL** (at 0 -12.2 90) (layer F.SilkS) hide
+      (effects (font (thickness 0.3048)))
+    )
+    (fp_line (start 15.24 3.81) (end 15.24 5.08) (layer F.SilkS) (width 0.381))
+    (fp_line (start 14.605 4.445) (end 15.875 4.445) (layer F.SilkS) (width 0.381))
+    (fp_circle (center 0 0) (end -1.27 -8.89) (layer F.SilkS) (width 0.20066))
+    (fp_circle (center 0 0) (end 6.35 8.89) (layer F.SilkS) (width 0.20066))
+    (pad 1 smd rect (at 15.485 0 90) (size 3.29 3.29) (layers F.Cu F.Paste F.Mask)
+      (net 37 +BATT))
+    (pad 2 smd rect (at -15.485 0 90) (size 3.29 3.29) (layers F.Cu F.Paste F.Mask)
+      (net 1 GND))
+    (model 3D/MPD_CR2032.wrl
+      (at (xyz 0 0 0))
+      (scale (xyz 0.3937 0.3937 0.3937))
+      (rotate (xyz 0 0 0))
+    )
+  )
+  (dimension 55.88 (width 0.3) (layer Dwgs.User)
+    (gr_text "55.880 mm" (at 125.65 121.92 270) (layer Dwgs.User)
+      (effects (font (size 1.5 1.5) (thickness 0.3)))
+    )
+    (feature1 (pts (xy 130.175 149.86) (xy 124.3 149.86)))
+    (feature2 (pts (xy 130.175 93.98) (xy 124.3 93.98)))
+    (crossbar (pts (xy 127 93.98) (xy 127 149.86)))
+    (arrow1a (pts (xy 127 149.86) (xy 126.413579 148.733496)))
+    (arrow1b (pts (xy 127 149.86) (xy 127.586421 148.733496)))
+    (arrow2a (pts (xy 127 93.98) (xy 126.413579 95.106504)))
+    (arrow2b (pts (xy 127 93.98) (xy 127.586421 95.106504)))
+  )
+  (dimension 95.885 (width 0.3) (layer Dwgs.User)
+    (gr_text "95.885 mm" (at 178.1175 90.725) (layer Dwgs.User)
+      (effects (font (size 1.5 1.5) (thickness 0.3)))
+    )
+    (feature1 (pts (xy 226.06 93.98) (xy 226.06 89.375)))
+    (feature2 (pts (xy 130.175 93.98) (xy 130.175 89.375)))
+    (crossbar (pts (xy 130.175 92.075) (xy 226.06 92.075)))
+    (arrow1a (pts (xy 226.06 92.075) (xy 224.933496 92.661421)))
+    (arrow1b (pts (xy 226.06 92.075) (xy 224.933496 91.488579)))
+    (arrow2a (pts (xy 130.175 92.075) (xy 131.301504 92.661421)))
+    (arrow2b (pts (xy 130.175 92.075) (xy 131.301504 91.488579)))
   )
   (gr_line (start 226.06 149.86) (end 226.06 93.98) (angle 90) (layer Edge.Cuts) (width 0.1))
@@
   (segment (start 153.035 105.75) (end 153.035 100.625) (width 0.25) (layer F.Cu) (net 33))
   (segment (start 151.435 105.75) (end 151.435 100.625) (width 0.25) (layer F.Cu) (net 34))
+  (segment (start 167.005 96.275) (end 167.005 103.505) (width 0.25) (layer F.Cu) (net 37))
+  (segment (start 169.037 104.013) (end 169.037 101.346) (width 0.25) (layer B.Cu) (net 37))
+  (segment (start 168.275 104.775) (end 169.037 104.013) (width 0.25) (layer B.Cu) (net 37))
+  (via (at 168.275 104.775) (size 0.6) (layers F.Cu B.Cu) (net 37))
+  (segment (start 167.005 103.505) (end 168.275 104.775) (width 0.25) (layer F.Cu) (net 37))
   (segment (start 146.574 121.92) (end 146.574 125) (width 0.25) (layer B.Cu) (net 39))
   (segment (start 146.574 125) (end 147.574 126) (width 0.25) (layer B.Cu) (net 39))
